File: PCB/VN-100 Breakout/VN-100Breakout/VN-100Breakout.kicad_pcb (KiCad board)
At the start: 2 copper layers, 6 parts

Commit message: Updated pin numbering on VN-100 Breakout symbol
Parts:
- moved X 287.4 mm to (271.8, 156.2)
- moved A 262.1 mm to (264.2, 180.3)
- moved REF** 221.9 mm to (203.2, 139.7), turned to 180 degrees
- moved VR 218.0 mm to (265.4, 132.1)
- moved U 210.2 mm to (221.0, 161.3)
- moved REF** 140.0 mm to (177.8, 151.1), turned to 180 degrees
