File: PCB/VN-100Breakout/VN-100Breakout.sch (KiCad schematic (older format))
At the start: 3 parts

Commit message: VN-100 Board Layout started
Parts:
- removed U?: VN-100, symbol PayloadSymbols:VN-100
- U1: renamed from U?; footprint (none) -> PayloadFootprints:VN-100Breakout
- U2: renamed from U?; footprint (none) -> PayloadFootprints:VN-100
Connections:
- wire segments 32 -> 36
Changed lines of the file:
@@
 $EndDescr
 $Comp
-L PayloadSymbols:VN-100_Breakout U?
+L PayloadSymbols:VN-100_Breakout U1
 U 1 1 6163BBA8
 P 4800 4000
-F 0 "U?" H 4800 4765 50  0000 C CNN
+F 0 "U1" H 4800 4765 50  0000 C CNN
 F 1 "VN-100_Breakout" H 4800 4674 50  0000 C CNN
-F 2 "" H 4850 4300 50  0001 C CNN
+F 2 "PayloadFootprints:VN-100Breakout" H 4850 4300 50  0001 C CNN
 F 3 "" H 4850 4300 50  0001 C CNN
 	1    4800 4000
@@
 $EndComp
 $Comp
-L PayloadSymbols:VN-100 U?
+L PayloadSymbols:VN-100 U2
 U 1 1 6163C870
 P 7400 4100
-F 0 "U?" H 7450 5331 50  0000 C CNN
+F 0 "U2" H 7450 5331 50  0000 C CNN
 F 1 "VN-100" H 7450 5240 50  0000 C CNN
-F 2 "" H 6600 4600 50  0001 C CNN
+F 2 "PayloadFootprints:VN-100" H 6600 4600 50  0001 C CNN
 F 3 "" H 6600 4600 50  0001 C CNN
 	1    7400 4100
@@
 Restore
 Wire Wire Line
-	5250 4100 5650 4100
-Text Label 5500 4100 0    50   ~ 0
+	5250 4250 5650 4250
+Text Label 5500 4250 0    50   ~ 0
 RX2
 Wire Wire Line
@@
 RX2
 Wire Wire Line
-	5250 4250 5650 4250
-Text Label 5500 4250 0    50   ~ 0
+	5250 4100 5650 4100
+Text Label 5500 4100 0    50   ~ 0
 TX2
 Wire Wire Line
@@
 GND
 Wire Wire Line
+	4350 3650 3950 3650
+Text Label 3950 3650 0    50   ~ 0
+RX1
+Wire Wire Line
+	7250 3050 7250 2650
+Text Label 7250 2800 1    50   ~ 0
+RX1
+Wire Wire Line
 	4350 3500 3950 3500
 Text Label 3950 3500 0    50   ~ 0
-RX1
+TX1
 Wire Wire Line
 	7500 3050 7500 2650
 Text Label 7500 2800 1    50   ~ 0
-RX1
-Wire Wire Line
-	4350 3650 3950 3650
-Text Label 3950 3650 0    50   ~ 0
-TX1
-Wire Wire Line
-	7250 3050 7250 2650
-Text Label 7250 2800 1    50   ~ 0
 TX1
 Wire Wire Line
@@
 Text Label 3950 3950 0    50   ~ 0
 SPI_MOSI
-$Comp
-L PayloadSymbols:VN-100 U?
-U 1 1 616483E5
-P 7400 4100
-F 0 "U?" H 7450 5331 50  0000 C CNN
-F 1 "VN-100" H 7450 5240 50  0000 C CNN
-F 2 "" H 6600 4600 50  0001 C CNN
-F 3 "" H 6600 4600 50  0001 C CNN
-	1    7400 4100
-	1    0    0    -1
-$EndComp
-Connection ~ 7950 3050
-Connection ~ 7750 3050
-Connection ~ 6250 3500
-Connection ~ 8650 4250
-Connection ~ 8650 4100
-Connection ~ 8650 3650
-Connection ~ 8200 3050
 Wire Wire Line
 	6250 3650 5850 3650
@@
 Wire Wire Line
 	6250 4250 5850 4250
-Connection ~ 6250 3950
-Connection ~ 7250 3050
-Connection ~ 7500 3050
 Text Label 5850 4250 0    50   ~ 0
 NRST
-Connection ~ 8650 3800
-Connection ~ 8650 3950
+Wire Wire Line
+	8650 4400 9050 4400
+Text Label 8900 4400 0    50   ~ 0
+GND
+Wire Wire Line
+	8650 4550 9050 4550
+Text Label 8900 4550 0    50   ~ 0
+GND
+Wire Wire Line
+	8200 4950 8200 5350
+Text Label 8200 5200 3    50   ~ 0
+GND
+Wire Wire Line
+	7750 4950 7750 5350
+Text Label 7750 5200 3    50   ~ 0
+GND
 $EndSCHEMATC
