File: PCB/VN-100Breakout/VN-100Breakout.kicad_pcb (KiCad board)
At the start: 2 copper layers, 36.1 x 33.5 mm, 2 parts, among them U1 VN-100_Breakout, U2 VN-100

Commit message: adjusted vn breakout
Parts:
- U2: footprint PayloadFootprints:VN-100 -> VN-100Breakout:VN-100
Changed lines of the file:
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@@
     (add_net "Net-(U2-Pad8)")
   )
-  (module VN-100Breakout:VN-100Breakout (layer Front)
-    (at 153.67 99.06)
-    (fp_text reference U1 (at 0 3.81) (layer F.SilkS) hide
-      (effects (font (size 1 1) (thickness 0.15)))
-    )
-    (fp_text value VN-100_Breakout (at 0 -16.51) (layer F.SilkS)
-      (effects (font (size 1 1) (thickness 0.15)))
-    )
-    (fp_line (start 17.78 15.24) (end 17.78 -17.78) (layer Dwgs.User) (width 0.12))
-    (fp_line (start -17.78 15.24) (end 17.78 15.24) (layer Dwgs.User) (width 0.12))
-    (fp_line (start -17.78 -17.78) (end -17.78 15.24) (layer Dwgs.User) (width 0.12))
-    (fp_line (start 17.78 -17.78) (end -17.78 -17.78) (layer Dwgs.User) (width 0.12))
-    (fp_poly (pts (xy 2 5.84) (xy -1.9 5.84) (xy -1.9 2.54) (xy 2 2.54)) (layer F.CrtYd) (width 0.1))
-    (pad "" thru_hole circle (at -15.24 12.7) (size 4 4) (drill 3) (layers *.Cu *.Mask))
-    (pad "" thru_hole circle (at 15.24 12.7) (size 4 4) (drill 3) (layers *.Cu *.Mask))
-    (pad "" thru_hole circle (at 15.24 -15.24 180) (size 4 4) (drill 3) (layers *.Cu *.Mask))
-    (pad "" thru_hole circle (at -15.24 -15.24) (size 4 4) (drill 3) (layers *.Cu *.Mask))
-    (pad 12 thru_hole circle (at 15.24 0) (size 1.524 1.524) (drill 0.762) (layers *.Cu *.Mask)
-      (net 14 /TX2))
-    (pad 11 thru_hole circle (at 15.24 2.54) (size 1.524 1.524) (drill 0.762) (layers *.Cu *.Mask)
-      (net 15 /RX2))
-    (pad 10 thru_hole circle (at 15.24 5.08) (size 1.524 1.524) (drill 0.762) (layers *.Cu *.Mask)
-      (net 13 /GND))
-    (pad 9 thru_hole circle (at 15.24 7.62) (size 1.524 1.524) (drill 0.762) (layers *.Cu *.Mask)
-      (net 13 /GND))
-    (pad 13 thru_hole circle (at 15.24 -2.54) (size 1.524 1.524) (drill 0.762) (layers *.Cu *.Mask)
-      (net 12 /Restore))
-    (pad 14 thru_hole circle (at 15.24 -5.08) (size 1.524 1.524) (drill 0.762) (layers *.Cu *.Mask)
-      (net 11 /SYNC_OUT))
-    (pad 15 thru_hole circle (at 15.24 -7.62) (size 1.524 1.524) (drill 0.762) (layers *.Cu *.Mask)
-      (net 10 /Vin))
-    (pad 16 thru_hole circle (at 15.24 -10.16) (size 1.524 1.524) (drill 0.762) (layers *.Cu *.Mask)
-      (net 9 /Enable))
-    (pad 1 thru_hole circle (at -15.24 -10.16) (size 1.524 1.524) (drill 0.762) (layers *.Cu *.Mask)
-      (net 5 /TX1))
-    (pad 8 thru_hole circle (at -15.24 7.62) (size 1.524 1.524) (drill 0.762) (layers *.Cu *.Mask)
-      (net 7 /SPI_CS))
-    (pad 5 thru_hole circle (at -15.24 0) (size 1.524 1.524) (drill 0.762) (layers *.Cu *.Mask)
-      (net 6 /SPI_MISO))
-    (pad 2 thru_hole circle (at -15.24 -7.62) (size 1.524 1.524) (drill 0.762) (layers *.Cu *.Mask)
-      (net 8 /RX1))
-    (pad 3 thru_hole circle (at -15.24 -5.08) (size 1.524 1.524) (drill 0.762) (layers *.Cu *.Mask)
-      (net 4 /SPI_SCK))
-    (pad 7 thru_hole circle (at -15.24 5.08) (size 1.524 1.524) (drill 0.762) (layers *.Cu *.Mask)
-      (net 3 /SYNC_IN))
-    (pad 6 thru_hole circle (at -15.24 2.54) (size 1.524 1.524) (drill 0.762) (layers *.Cu *.Mask)
-      (net 2 /NRST))
-    (pad 4 thru_hole circle (at -15.24 -2.54) (size 1.524 1.524) (drill 0.762) (layers *.Cu *.Mask)
-      (net 1 /SPI_MOSI))
-  )
-  (module PayloadFootprints:VN-100 (layer Front)
+  (module VN-100Breakout:VN-100 (layer Front)
     (at 153.67 97.79)
     (fp_text reference U2 (at 0 -3.81) (layer F.SilkS) hide
@@
       (effects (font (size 1 1) (thickness 0.15)))
     )
+    (fp_poly (pts (xy 0.2 0.2) (xy -0.2 0.2) (xy -0.2 -0.2) (xy 0.2 -0.2)) (layer F.CrtYd) (width 0.1))
+    (fp_line (start -12.065 -13.335) (end 12.065 -13.335) (layer F.SilkS) (width 0.12))
+    (fp_line (start 12.065 -13.335) (end 12.065 13.335) (layer F.SilkS) (width 0.12))
+    (fp_line (start 12.065 13.335) (end -12.065 13.335) (layer F.SilkS) (width 0.12))
     (fp_line (start -12.065 13.335) (end -12.065 -13.335) (layer F.SilkS) (width 0.12))
-    (fp_line (start 12.065 13.335) (end -12.065 13.335) (layer F.SilkS) (width 0.12))
-    (fp_line (start 12.065 -13.335) (end 12.065 13.335) (layer F.SilkS) (width 0.12))
-    (fp_line (start -12.065 -13.335) (end 12.065 -13.335) (layer F.SilkS) (width 0.12))
-    (fp_line (start -12.192 13.462) (end -12.192 -13.462) (layer F.CrtYd) (width 0.12))
-    (fp_line (start 12.192 -13.462) (end 12.192 13.462) (layer F.CrtYd) (width 0.12))
-    (fp_line (start 12.192 13.462) (end -12.192 13.462) (layer F.CrtYd) (width 0.12))
-    (fp_line (start 12.192 -13.462) (end -12.192 -13.462) (layer F.CrtYd) (width 0.12))
     (pad 16 smd rect (at -10.287 -8.89 90) (size 1.143 2.54) (layers Front F.Paste F.Mask)
       (net 4 /SPI_SCK))
@@
     (pad 9 smd rect (at 7.62 -11.303) (size 1.143 2.54) (layers Front F.Paste F.Mask)
       (net 11 /SYNC_OUT))
+    (model "C:/Users/raidr/Documents/Programming/LBR/Payload-2022-Electrical/PCB/Library/Step Files/vn100_smd.step"
+      (offset (xyz -11 -12 1))
+      (scale (xyz 1 1 1))
+      (rotate (xyz 0 180 90))
+    )
+  )
+  (module VN-100Breakout:VN-100Breakout (layer Front)
+    (at 153.67 99.06)
+    (fp_text reference U1 (at 0 3.81) (layer F.SilkS) hide
+      (effects (font (size 1 1) (thickness 0.15)))
+    )
+    (fp_text value VN-100_Breakout (at 0 -16.51) (layer F.SilkS)
+      (effects (font (size 1 1) (thickness 0.15)))
+    )
+    (fp_line (start 17.78 15.24) (end 17.78 -17.78) (layer Dwgs.User) (width 0.12))
+    (fp_line (start -17.78 15.24) (end 17.78 15.24) (layer Dwgs.User) (width 0.12))
+    (fp_line (start -17.78 -17.78) (end -17.78 15.24) (layer Dwgs.User) (width 0.12))
+    (fp_line (start 17.78 -17.78) (end -17.78 -17.78) (layer Dwgs.User) (width 0.12))
+    (fp_poly (pts (xy 2 5.84) (xy -1.9 5.84) (xy -1.9 2.54) (xy 2 2.54)) (layer F.CrtYd) (width 0.1))
+    (pad "" thru_hole circle (at -15.24 12.7) (size 4 4) (drill 3) (layers *.Cu *.Mask))
+    (pad "" thru_hole circle (at 15.24 12.7) (size 4 4) (drill 3) (layers *.Cu *.Mask))
+    (pad "" thru_hole circle (at 15.24 -15.24 180) (size 4 4) (drill 3) (layers *.Cu *.Mask))
+    (pad "" thru_hole circle (at -15.24 -15.24) (size 4 4) (drill 3) (layers *.Cu *.Mask))
+    (pad 12 thru_hole circle (at 15.24 0) (size 1.524 1.524) (drill 0.762) (layers *.Cu *.Mask)
+      (net 14 /TX2))
+    (pad 11 thru_hole circle (at 15.24 2.54) (size 1.524 1.524) (drill 0.762) (layers *.Cu *.Mask)
+      (net 15 /RX2))
+    (pad 10 thru_hole circle (at 15.24 5.08) (size 1.524 1.524) (drill 0.762) (layers *.Cu *.Mask)
+      (net 13 /GND))
+    (pad 9 thru_hole circle (at 15.24 7.62) (size 1.524 1.524) (drill 0.762) (layers *.Cu *.Mask)
+      (net 13 /GND))
+    (pad 13 thru_hole circle (at 15.24 -2.54) (size 1.524 1.524) (drill 0.762) (layers *.Cu *.Mask)
+      (net 12 /Restore))
+    (pad 14 thru_hole circle (at 15.24 -5.08) (size 1.524 1.524) (drill 0.762) (layers *.Cu *.Mask)
+      (net 11 /SYNC_OUT))
+    (pad 15 thru_hole circle (at 15.24 -7.62) (size 1.524 1.524) (drill 0.762) (layers *.Cu *.Mask)
+      (net 10 /Vin))
+    (pad 16 thru_hole circle (at 15.24 -10.16) (size 1.524 1.524) (drill 0.762) (layers *.Cu *.Mask)
+      (net 9 /Enable))
+    (pad 1 thru_hole circle (at -15.24 -10.16) (size 1.524 1.524) (drill 0.762) (layers *.Cu *.Mask)
+      (net 5 /TX1))
+    (pad 8 thru_hole circle (at -15.24 7.62) (size 1.524 1.524) (drill 0.762) (layers *.Cu *.Mask)
+      (net 7 /SPI_CS))
+    (pad 5 thru_hole circle (at -15.24 0) (size 1.524 1.524) (drill 0.762) (layers *.Cu *.Mask)
+      (net 6 /SPI_MISO))
+    (pad 2 thru_hole circle (at -15.24 -7.62) (size 1.524 1.524) (drill 0.762) (layers *.Cu *.Mask)
+      (net 8 /RX1))
+    (pad 3 thru_hole circle (at -15.24 -5.08) (size 1.524 1.524) (drill 0.762) (layers *.Cu *.Mask)
+      (net 4 /SPI_SCK))
+    (pad 7 thru_hole circle (at -15.24 5.08) (size 1.524 1.524) (drill 0.762) (layers *.Cu *.Mask)
+      (net 3 /SYNC_IN))
+    (pad 6 thru_hole circle (at -15.24 2.54) (size 1.524 1.524) (drill 0.762) (layers *.Cu *.Mask)
+      (net 2 /NRST))
+    (pad 4 thru_hole circle (at -15.24 -2.54) (size 1.524 1.524) (drill 0.762) (layers *.Cu *.Mask)
+      (net 1 /SPI_MOSI))
   )
   (gr_poly (pts (xy 176.53 116.84) (xy 130.81 116.84) (xy 130.81 78.74) (xy 176.53 78.74)) (layer Cmts.User) (width 0.1))
