File: PCB/VN-100Breakout/VN-100Breakout.kicad_pcb (KiCad board)
At the start: 2 copper layers, 36.1 x 33.5 mm, 2 parts, among them U1 VN-100_Breakout, U2 VN-100

Commit message: credits
Other:
- board text added: "Created By: Josias Navasca Aiden Little Martin Lee Anthony Le"
Changed lines of the file:
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@@
   (general
     (thickness 1.6002)
-    (drawings 28)
+    (drawings 29)
     (tracks 82)
     (zones 0)
@@
       (effects (font (size 1 1) (thickness 0.15)))
     )
+    (fp_line (start -12.065 13.335) (end -12.065 -13.335) (layer F.SilkS) (width 0.12))
+    (fp_line (start 12.065 13.335) (end -12.065 13.335) (layer F.SilkS) (width 0.12))
+    (fp_line (start 12.065 -13.335) (end 12.065 13.335) (layer F.SilkS) (width 0.12))
+    (fp_line (start -12.065 -13.335) (end 12.065 -13.335) (layer F.SilkS) (width 0.12))
     (fp_poly (pts (xy 0.2 0.2) (xy -0.2 0.2) (xy -0.2 -0.2) (xy 0.2 -0.2)) (layer F.CrtYd) (width 0.1))
-    (fp_line (start -12.065 -13.335) (end 12.065 -13.335) (layer F.SilkS) (width 0.12))
-    (fp_line (start 12.065 -13.335) (end 12.065 13.335) (layer F.SilkS) (width 0.12))
-    (fp_line (start 12.065 13.335) (end -12.065 13.335) (layer F.SilkS) (width 0.12))
-    (fp_line (start -12.065 13.335) (end -12.065 -13.335) (layer F.SilkS) (width 0.12))
     (pad 16 smd rect (at -10.287 -8.89 90) (size 1.143 2.54) (layers Front F.Paste F.Mask)
       (net 4 /SPI_SCK))
@@
       (effects (font (size 1 1) (thickness 0.15)))
     )
+    (fp_poly (pts (xy 2 5.84) (xy -1.9 5.84) (xy -1.9 2.54) (xy 2 2.54)) (layer F.CrtYd) (width 0.1))
+    (fp_line (start 17.78 -17.78) (end -17.78 -17.78) (layer Dwgs.User) (width 0.12))
+    (fp_line (start -17.78 -17.78) (end -17.78 15.24) (layer Dwgs.User) (width 0.12))
+    (fp_line (start -17.78 15.24) (end 17.78 15.24) (layer Dwgs.User) (width 0.12))
     (fp_line (start 17.78 15.24) (end 17.78 -17.78) (layer Dwgs.User) (width 0.12))
-    (fp_line (start -17.78 15.24) (end 17.78 15.24) (layer Dwgs.User) (width 0.12))
-    (fp_line (start -17.78 -17.78) (end -17.78 15.24) (layer Dwgs.User) (width 0.12))
-    (fp_line (start 17.78 -17.78) (end -17.78 -17.78) (layer Dwgs.User) (width 0.12))
-    (fp_poly (pts (xy 2 5.84) (xy -1.9 5.84) (xy -1.9 2.54) (xy 2 2.54)) (layer F.CrtYd) (width 0.1))
     (pad "" thru_hole circle (at -15.24 12.7) (size 4 4) (drill 3) (layers *.Cu *.Mask))
     (pad "" thru_hole circle (at 15.24 12.7) (size 4 4) (drill 3) (layers *.Cu *.Mask))
@@
     (pad 4 thru_hole circle (at -15.24 -2.54) (size 1.524 1.524) (drill 0.762) (layers *.Cu *.Mask)
       (net 1 /SPI_MOSI))
+  )
+  (gr_text "Created By:\nJosias Navasca\nAiden Little\nMartin Lee\nAnthony Le\n" (at 154.305 86.36) (layer B.SilkS)
+    (effects (font (size 0.8128 0.8128) (thickness 0.1524)) (justify mirror))
   )
   (gr_line (start 148.867813 98.725037) (end 151.272876 94.548325) (layer F.SilkS) (width 0.28125))
@@
     (polygon
       (pts
-        (xy 176.53 116.84) (xy 130.81 116.84) (xy 130.81 78.74) (xy 176.53 78.74)
+        (xy 172.72 116.84) (xy 134.62 116.84) (xy 134.62 78.74) (xy 172.72 78.74)
       )
     )
