File: PCB/DevelopmentBoard/DevelopmentBoard.sch (KiCad schematic (older format))
At the start: 20 parts, among them J1 Conn_01x04_MountingPin, U1 Pi_CM4, U2 Barometer_Grove, U3 D24V22F5, U4 Micro-USB, U5 VN-100_Breakout, X1 XT30-M_Connector, X2 XT30-M_Connector, X3 2mmGrove_Connector

Commit message: Removed "PayloadSymbols" Folder, consolidated symbols and footprints into DevelopmentBoard Folder
Parts:
- A1: symbol PayloadSymbols:TBS_Crossfire_RF -> DevelopmentBoard:TBS_Crossfire_RF
- J1: symbol PayloadSymbols:Conn_01x04_MountingPin -> DevelopmentBoard-rescue:Conn_01x04_MountingPin-PayloadSymbols
- U1: symbol PayloadSymbols:Pi_CM4 -> DevelopmentBoard:Pi_CM4
- U1: symbol PayloadSymbols:Pi_CM4 -> DevelopmentBoard-rescue:Pi_CM4-PayloadSymbols
- U2: symbol PayloadSymbols:Barometer_Grove -> DevelopmentBoard-rescue:Barometer_Grove-PayloadSymbols
- U3: symbol PayloadSymbols:D24V22F5 -> DevelopmentBoard:D24V22F5
- U4: symbol PayloadSymbols:Micro-USB -> DevelopmentBoard:Micro-USB
- U5: symbol PayloadSymbols:VN-100_Breakout -> DevelopmentBoard:VN-100_Breakout
- X1, X2: symbol PayloadSymbols:XT30-M_Connector -> DevelopmentBoard-rescue:XT30-M_Connector-PayloadSymbols
- X3: symbol PayloadSymbols:2mmGrove_Connector -> DevelopmentBoard:2mmGrove_Connector
Changed lines of the file:
@@
 $EndDescr
 $Comp
-L PayloadSymbols:Pi_CM4 U1
+L DevelopmentBoard:Pi_CM4 U1
 U 1 1 615FC623
 P 8150 4250
@@
 $EndComp
 $Comp
-L PayloadSymbols:Pi_CM4 U1
+L DevelopmentBoard-rescue:Pi_CM4-PayloadSymbols U1
 U 2 1 6160B108
 P 13400 4250
@@
 $EndComp
 $Comp
-L PayloadSymbols:D24V22F5 U3
+L DevelopmentBoard:D24V22F5 U3
 U 1 1 61620546
 P 18900 2750
@@
 $EndComp
 $Comp
-L PayloadSymbols:TBS_Crossfire_RF A1
+L DevelopmentBoard:TBS_Crossfire_RF A1
 U 1 1 616210FE
 P 19250 7500
@@
 $EndComp
 $Comp
-L PayloadSymbols:Micro-USB U4
+L DevelopmentBoard:Micro-USB U4
 U 1 1 6166969C
 P 19150 8700
@@
 $EndComp
 $Comp
-L PayloadSymbols:2mmGrove_Connector X3
+L DevelopmentBoard:2mmGrove_Connector X3
 U 1 1 61667DE2
 P 18300 6300
@@
 $EndComp
 $Comp
-L PayloadSymbols:Barometer_Grove U2
+L DevelopmentBoard-rescue:Barometer_Grove-PayloadSymbols U2
 U 1 1 6168942A
 P 19600 6250
@@
 $EndComp
 $Comp
-L PayloadSymbols:VN-100_Breakout U5
+L DevelopmentBoard:VN-100_Breakout U5
 U 1 1 61690F0C
 P 19300 4900
@@
 CH1
 $Comp
-L PayloadSymbols:XT30-M_Connector X1
+L DevelopmentBoard-rescue:XT30-M_Connector-PayloadSymbols X1
 U 1 1 617175F8
 P 18000 2250
@@
 	18250 2200 18150 2200
 $Comp
-L PayloadSymbols:XT30-M_Connector X2
+L DevelopmentBoard-rescue:XT30-M_Connector-PayloadSymbols X2
 U 1 1 6171A8B5
 P 18100 2650
@@
 $EndComp
 $Comp
-L PayloadSymbols:Conn_01x04_MountingPin J1
+L DevelopmentBoard-rescue:Conn_01x04_MountingPin-PayloadSymbols J1
 U 1 1 6180C683
 P 20850 5150

Commit message: Added USB Controller symbol, footprint, and Step File
Parts:
- added IC?: FE1.1S_USB_Controller, SOP64P600X175-28N, symbol DevelopmentBoard:FE1.1S_USB_Controller
- added R2, R4: 0, DevelopmentBoard:0603, symbol Device:R_Small_US
- R10, R7, R8, R9: footprint PayloadFootprints:0603 -> DevelopmentBoard:0603
Connections:
- wire segments 59 -> 61
Changed lines of the file:
@@
 D+
 Wire Wire Line
-	18950 8650 18650 8650
-Text Label 18650 8650 0    50   ~ 0
+	18500 8650 18200 8650
+Text Label 18200 8650 0    50   ~ 0
 D-
 Wire Wire Line
-	18950 8750 18650 8750
-Text Label 18650 8750 0    50   ~ 0
+	18500 8750 18200 8750
+Text Label 18200 8750 0    50   ~ 0
 D+
 $Comp
@@
 F 0 "R10" H 19918 4446 50  0000 L CNN
 F 1 "0" H 19918 4355 50  0000 L CNN
-F 2 "PayloadFootprints:0603" H 19850 4400 50  0001 C CNN
+F 2 "DevelopmentBoard:0603" H 19850 4400 50  0001 C CNN
 F 3 "~" H 19850 4400 50  0001 C CNN
 	1    19850 4400
@@
 F 0 "R9" V 18818 4596 50  0000 L CNN
 F 1 "0" V 18818 4505 50  0000 L CNN
-F 2 "PayloadFootprints:0603" H 18750 4550 50  0001 C CNN
+F 2 "DevelopmentBoard:0603" H 18750 4550 50  0001 C CNN
 F 3 "~" H 18750 4550 50  0001 C CNN
 	1    18750 4550
@@
 F 0 "R8" V 18818 4446 50  0000 L CNN
 F 1 "0" V 18818 4355 50  0000 L CNN
-F 2 "PayloadFootprints:0603" H 18750 4400 50  0001 C CNN
+F 2 "DevelopmentBoard:0603" H 18750 4400 50  0001 C CNN
 F 3 "~" H 18750 4400 50  0001 C CNN
 	1    18750 4400
@@
 F 0 "R7" V 18618 5196 50  0000 L CNN
 F 1 "0" V 18618 5105 50  0000 L CNN
-F 2 "PayloadFootprints:0603" H 18550 5150 50  0001 C CNN
+F 2 "DevelopmentBoard:0603" H 18550 5150 50  0001 C CNN
 F 3 "~" H 18550 5150 50  0001 C CNN
 	1    18550 5150
@@
 Wire Wire Line
 	8150 8950 8000 8950
+$Comp
+L Device:R_Small_US R4
+U 1 1 61A8FCC8
+P 18600 8750
+F 0 "R4" V 18668 8796 50  0000 L CNN
+F 1 "0" V 18668 8705 50  0000 L CNN
+F 2 "DevelopmentBoard:0603" H 18600 8750 50  0001 C CNN
+F 3 "~" H 18600 8750 50  0001 C CNN
+	1    18600 8750
+	0    -1   -1   0
+$EndComp
+$Comp
+L Device:R_Small_US R2
+U 1 1 61A8FCCE
+P 18600 8650
+F 0 "R2" V 18668 8696 50  0000 L CNN
+F 1 "0" V 18668 8605 50  0000 L CNN
+F 2 "DevelopmentBoard:0603" H 18600 8650 50  0001 C CNN
+F 3 "~" H 18600 8650 50  0001 C CNN
+	1    18600 8650
+	0    -1   -1   0
+$EndComp
+$Comp
+L DevelopmentBoard:FE1.1S_USB_Controller IC?
+U 1 1 61AA4FD8
+P 18300 10350
+F 0 "IC?" H 18950 10615 50  0000 C CNN
+F 1 "FE1.1S_USB_Controller" H 18950 10524 50  0000 C CNN
+F 2 "SOP64P600X175-28N" H 19450 10450 50  0001 L CNN
+F 3 "https://cdn-shop.adafruit.com/product-files/2991/FE1.1s+Data+Sheet+(Rev.+1.0).pdf" H 20600 10250 50  0001 L CNN
+F 4 "1.75" H 19450 10150 50  0001 L CNN "Height"
+F 5 "JFD IC" H 19450 10050 50  0001 L CNN "Manufacturer_Name"
+F 6 "FE1.1S" H 19450 9950 50  0001 L CNN "Manufacturer_Part_Number"
+	1    18300 10350
+	1    0    0    -1
+$EndComp
+Wire Wire Line
+	18700 8650 18950 8650
+Wire Wire Line
+	18700 8750 18950 8750
 $EndSCHEMATC
