File: PCB/DevelopmentBoard/_autosave-DevelopmentBoard.sch (KiCad schematic (older format))
At the start: 28 parts, among them J1 Conn_01x04_MountingPin, J2 Conn_01x04_MountingPin-Payloa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, J5 Conn_01x04_MountingPin, U1 D24V22F5_VoltageRegulator, U2 Barometer_Grove, U3 RASPBERRY_PI_3_MODEL_B+, U4 Conn_01x08_DevBoardSymbols, U6 MCP3008_ADC, U7 Conn_01x06_DevBoard_Symbols, X1 XT30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

Commit message: Revert "Merge branch 'main' of https://github.com/CSULB-LBR/Payload-2022-Electrical"
This reverts commit 36186b0aa135225f420ab8312ad97e4f675c68a7, reversing
changes made to 173b9dac6d612d33aa589f2b9774fff44ddaf61c.
Parts:
- R20: renamed from R12; footprint (none) -> DevelopmentBoard:0603
Changed lines of the file:
@@
 $EndComp
 $Comp
-L Device:R_Small_US R12
+L Device:R_Small_US R20
 U 1 1 626DE972
 P 1150 17100
-F 0 "R12" H 1218 17146 50  0000 L CNN
+F 0 "R20" H 1218 17146 50  0000 L CNN
 F 1 "4.7k" H 1218 17055 50  0000 L CNN
-F 2 "" H 1150 17100 50  0001 C CNN
+F 2 "DevelopmentBoard:0603" H 1150 17100 50  0001 C CNN
 F 3 "~" H 1150 17100 50  0001 C CNN
 	1    1150 17100
@@
 $EndComp
 $Comp
-L power:+3.3V #PWR?
+L power:+3.3V #PWR0115
 U 1 1 626DFEE0
 P 1150 17000
-F 0 "#PWR?" H 1150 16850 50  0001 C CNN
+F 0 "#PWR0115" H 1150 16850 50  0001 C CNN
 F 1 "+3.3V" H 1165 17173 50  0000 C CNN
 F 2 "" H 1150 17000 50  0001 C CNN

Commit message: Routed signal traces from ADC to Crossfire receiver
Connections:
- net labels removed: VN-100_CS
Changed lines of the file:
@@
 $EndComp
 Text Label 2400 17900 1    50   ~ 0
-VN-100_CS
+VIN-100_CS
 $Comp
 L power:+3.3V #PWR0163
@@
 SDA
 Text Label 4800 15700 2    50   ~ 0
+CH0
+Text Label 4800 15800 2    50   ~ 0
 CH1
-Text Label 4800 15800 2    50   ~ 0
-CH2
 $Comp
 L DevelopmentBoard-rescue:XT30-M_Connector-PayloadSymbols X1
@@
 	4400 15900 4800 15900
 Text Label 4650 15900 0    50   ~ 0
-CH3
+CH2
 Wire Wire Line
 	4400 16000 4800 16000
 Text Label 4650 16000 0    50   ~ 0
-CH4
+CH3
 Wire Wire Line
 	4400 16100 4800 16100
 Text Label 4650 16100 0    50   ~ 0
-CH5
+CH4
 Wire Wire Line
 	3600 16000 3200 16000
@@
 	3600 16100 3200 16100
 Text Label 3200 16100 0    50   ~ 0
+CH5
+Text Label 3200 16000 0    50   ~ 0
 CH6
-Text Label 3200 16000 0    50   ~ 0
-CH7
 Text Label 3200 15900 0    50   ~ 0
 CH7
@@
 Wire Wire Line
 	6250 3050 6550 3050
-Wire Wire Line
-	1950 4250 1750 4250
-Wire Wire Line
-	1950 4350 1750 4350
-Text Label 1800 4250 0    50   ~ 0
-SDA
-Text Label 1800 4350 0    50   ~ 0
-SCL
 Text Label 1500 3650 0    50   ~ 0
 VIN-100_CS
@@
 Text Label 1150 17900 1    50   ~ 0
 CS_SHDN
+Text Label 1800 4350 0    50   ~ 0
+SCL
+Text Label 1800 4250 0    50   ~ 0
+SDA
+Wire Wire Line
+	1950 4350 1750 4350
+Wire Wire Line
+	1950 4250 1750 4250
 $EndSCHEMATC
