File: PCB/DevelopmentBoard/_autosave-DevelopmentBoard.kicad_pcb (KiCad board)
At the start: 2 copper layers, 152.4 x 76.2 mm, 51 parts, among them J1 Conn_01x04_MountingPin, J2 Conn_01x04_MountingPin-Payloa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, J5 Conn_01x04_MountingPin, U1 D24V22F5_VoltageRegulator, U3 RASPBERRY_PI_3_MODEL_B+, U4 Conn_01x08_DevBoardSymbols, U6 MCP3008_ADC, U7 Conn_01x06_DevBoard_Symbols, X1 XT30, X2 XT30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

Commit message: Revert "Merge branch 'main' of https://github.com/CSULB-LBR/Payload-2022-Electrical"
This reverts commit 36186b0aa135225f420ab8312ad97e4f675c68a7, reversing
changes made to 173b9dac6d612d33aa589f2b9774fff44ddaf61c.
Parts:
- removed R12, R13, R14, R15: 0, DevelopmentBoard:0603
Changed lines of the file:
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@@
     (tracks 0)
     (zones 0)
-    (modules 51)
+    (modules 47)
     (nets 75)
   )
@@
   )
   (module DevelopmentBoard:0603 (layer Front)
-    (at 128.014001 153.730001)
-    (fp_text reference R12 (at 0 -5.715) (layer F.SilkS)
-      (effects (font (size 1 1) (thickness 0.15)))
-    )
-    (fp_text value 0 (at 0 5.08) (layer F.Fab)
-      (effects (font (size 1 1) (thickness 0.15)))
-    )
-    (fp_line (start -1.2 -0.6) (end -1.2 0.6) (layer F.SilkS) (width 0.12))
-    (fp_line (start -1.2 0.6) (end 1.2 0.6) (layer F.SilkS) (width 0.12))
-    (fp_line (start 1.2 0.6) (end 1.2 -0.6) (layer F.SilkS) (width 0.12))
-    (fp_line (start 1.2 -0.6) (end -1.2 -0.6) (layer F.SilkS) (width 0.12))
-    (fp_line (start -1.4 -0.8) (end 1.4 -0.8) (layer F.CrtYd) (width 0.12))
-    (fp_line (start 1.4 -0.8) (end 1.4 0.8) (layer F.CrtYd) (width 0.12))
-    (fp_line (start 1.4 0.8) (end -1.4 0.8) (layer F.CrtYd) (width 0.12))
-    (fp_line (start -1.4 0.8) (end -1.4 -0.8) (layer F.CrtYd) (width 0.12))
-    (pad 1 smd rect (at -0.75 0) (size 0.6 0.9) (layers Front F.Paste F.Mask)
-      (net 8 /CH4))
-    (pad 2 smd rect (at 0.75 0) (size 0.6 0.9) (layers Front F.Paste F.Mask)
-      (net 62 "Net-(R12-Pad2)"))
-    (model ${KIPRJMOD}/Models/Resistor_0603_Text.step
-      (at (xyz 0 0 0))
-      (scale (xyz 1 1 1))
-      (rotate (xyz 0 0 0))
-    )
-  )
-  (module DevelopmentBoard:0603 (layer Front)
-    (at 128.014001 156.450001)
-    (fp_text reference R13 (at 0 -5.715) (layer F.SilkS)
-      (effects (font (size 1 1) (thickness 0.15)))
-    )
-    (fp_text value 0 (at 0 5.08) (layer F.Fab)
-      (effects (font (size 1 1) (thickness 0.15)))
-    )
-    (fp_line (start -1.4 0.8) (end -1.4 -0.8) (layer F.CrtYd) (width 0.12))
-    (fp_line (start 1.4 0.8) (end -1.4 0.8) (layer F.CrtYd) (width 0.12))
-    (fp_line (start 1.4 -0.8) (end 1.4 0.8) (layer F.CrtYd) (width 0.12))
-    (fp_line (start -1.4 -0.8) (end 1.4 -0.8) (layer F.CrtYd) (width 0.12))
-    (fp_line (start 1.2 -0.6) (end -1.2 -0.6) (layer F.SilkS) (width 0.12))
-    (fp_line (start 1.2 0.6) (end 1.2 -0.6) (layer F.SilkS) (width 0.12))
-    (fp_line (start -1.2 0.6) (end 1.2 0.6) (layer F.SilkS) (width 0.12))
-    (fp_line (start -1.2 -0.6) (end -1.2 0.6) (layer F.SilkS) (width 0.12))
-    (pad 2 smd rect (at 0.75 0) (size 0.6 0.9) (layers Front F.Paste F.Mask)
-      (net 61 "Net-(R13-Pad2)"))
-    (pad 1 smd rect (at -0.75 0) (size 0.6 0.9) (layers Front F.Paste F.Mask)
-      (net 10 /CH5))
-    (model ${KIPRJMOD}/Models/Resistor_0603_Text.step
-      (at (xyz 0 0 0))
-      (scale (xyz 1 1 1))
-      (rotate (xyz 0 0 0))
-    )
-  )
-  (module DevelopmentBoard:0603 (layer Front)
-    (at 131.934001 153.730001)
-    (fp_text reference R14 (at 0 -5.715) (layer F.SilkS)
-      (effects (font (size 1 1) (thickness 0.15)))
-    )
-    (fp_text value 0 (at 0 5.08) (layer F.Fab)
-      (effects (font (size 1 1) (thickness 0.15)))
-    )
-    (fp_line (start -1.2 -0.6) (end -1.2 0.6) (layer F.SilkS) (width 0.12))
-    (fp_line (start -1.2 0.6) (end 1.2 0.6) (layer F.SilkS) (width 0.12))
-    (fp_line (start 1.2 0.6) (end 1.2 -0.6) (layer F.SilkS) (width 0.12))
-    (fp_line (start 1.2 -0.6) (end -1.2 -0.6) (layer F.SilkS) (width 0.12))
-    (fp_line (start -1.4 -0.8) (end 1.4 -0.8) (layer F.CrtYd) (width 0.12))
-    (fp_line (start 1.4 -0.8) (end 1.4 0.8) (layer F.CrtYd) (width 0.12))
-    (fp_line (start 1.4 0.8) (end -1.4 0.8) (layer F.CrtYd) (width 0.12))
-    (fp_line (start -1.4 0.8) (end -1.4 -0.8) (layer F.CrtYd) (width 0.12))
-    (pad 1 smd rect (at -0.75 0) (size 0.6 0.9) (layers Front F.Paste F.Mask)
-      (net 12 /CH6))
-    (pad 2 smd rect (at 0.75 0) (size 0.6 0.9) (layers Front F.Paste F.Mask)
-      (net 60 "Net-(R14-Pad2)"))
-    (model ${KIPRJMOD}/Models/Resistor_0603_Text.step
-      (at (xyz 0 0 0))
-      (scale (xyz 1 1 1))
-      (rotate (xyz 0 0 0))
-    )
-  )
-  (module DevelopmentBoard:0603 (layer Front)
-    (at 131.934001 156.450001)
-    (fp_text reference R15 (at 0 -5.715) (layer F.SilkS)
-      (effects (font (size 1 1) (thickness 0.15)))
-    )
-    (fp_text value 0 (at 0 5.08) (layer F.Fab)
-      (effects (font (size 1 1) (thickness 0.15)))
-    )
-    (fp_line (start -1.4 0.8) (end -1.4 -0.8) (layer F.CrtYd) (width 0.12))
-    (fp_line (start 1.4 0.8) (end -1.4 0.8) (layer F.CrtYd) (width 0.12))
-    (fp_line (start 1.4 -0.8) (end 1.4 0.8) (layer F.CrtYd) (width 0.12))
-    (fp_line (start -1.4 -0.8) (end 1.4 -0.8) (layer F.CrtYd) (width 0.12))
-    (fp_line (start 1.2 -0.6) (end -1.2 -0.6) (layer F.SilkS) (width 0.12))
-    (fp_line (start 1.2 0.6) (end 1.2 -0.6) (layer F.SilkS) (width 0.12))
-    (fp_line (start -1.2 0.6) (end 1.2 0.6) (layer F.SilkS) (width 0.12))
-    (fp_line (start -1.2 -0.6) (end -1.2 0.6) (layer F.SilkS) (width 0.12))
-    (pad 2 smd rect (at 0.75 0) (size 0.6 0.9) (layers Front F.Paste F.Mask)
-      (net 59 "Net-(R15-Pad2)"))
-    (pad 1 smd rect (at -0.75 0) (size 0.6 0.9) (layers Front F.Paste F.Mask)
-      (net 11 /CH7))
-    (model ${KIPRJMOD}/Models/Resistor_0603_Text.step
-      (at (xyz 0 0 0))
-      (scale (xyz 1 1 1))
-      (rotate (xyz 0 0 0))
-    )
-  )
-  (module DevelopmentBoard:0603 (layer Front)
