File: Recovery PCB/GPS Board/GPS_Board/_autosave-GPS_Board.kicad_sch (KiCad schematic)
At the start: 11 parts

Commit message: XBEE Labels
Parts:
- A1: value (none) -> XBee-3-Pro; footprint (none) -> GPS Board:XBEE-20_THT
- A2: value (none) -> Sparkfun-GPS-Breakout; footprint (none) -> GPS Board:Sparkfun-GPS-ZOE-M8Q-Breakout
- A3: value (none) -> Eboot-MP1584EN-5V-Power-Supply; footprint (none) -> GPS Board:EBOOT-MP1584EN-5N-POWER-SUPPLY
- J1, J2: value (none) -> XT30-M; footprint (none) -> Connector_AMASS:AMASS_XT30U-M_1x02_P5.0mm_Vertical
- TP1, TP2, TP3, TP4: value (none) -> TestPoint; footprint (none) -> TestPoint:TestPoint_Pad_D1.5mm
- TP5: value (none) -> TestPoint; footprint (none) -> TestPoint:TestPoint_Pad_D1.0mm
- U1: value (none) -> Teensy4.1; footprint (none) -> GPS Board:Teensy41
Connections:
- net AD3/SPI_SSEL: now reaches A1.17 (AD3/SPI_SSEL), U1.12 (10_CS_MQSR)
- net SPI_MISO: now reaches A1.4 (SPI_MISO), U1.14 (12_MISO_MQSL)
- net ON/SLEEP_XBEE: now reaches A1.13 (ON/SLEEP), U1.25 (33_MCLK2)
- net RESET_XBEE: now reaches A1.5 (RESET), U1.29 (37_CS)
- net DTR_XBEE: now reaches A1.9 (DTR), U1.30 (38_CS1_IN1)
- net AD2/SPI_CLOCK: now reaches A1.18 (AD2/SPI_CLOCK), U1.35 (13_SCK_LED)
- net RSSI_PWM: now reaches A1.6 (RSSI_PWM), U1.44 (22_A8_CTX1)
